Commit message: Added two links with variable buoyancy. Some changes to fluid plugin.

File: urdf/uauv.xacro (robot description, xacro)
@@ -7,8 +7,33 @@
   <xacro:property name="body_length"      value="0.667"/>
   <xacro:property name="X_cog"            value="-0.55"/>
+  <!-- Variable buoyancy link -->
+  <xacro:macro name="buoyancy_link" params="name xyz">
+    <joint name="${name}" type="revolute">
+      <parent link="base_link"/>
+      <child link="${name}"/>
+      <origin rpy="0 0 0" xyz="${xyz}"/>
+      <axis xyz="0 1 0"/>
+      <limit effort="0" velocity="5.0" lower="0" upper="0" />
+    </joint>
+    <link name="${name}">
+      <buoyancy>
+        <variable compensation="3.0"/>
+      </buoyancy>
+      <inertial>
+        <mass value=".1"/>
+        <inertia
+          ixx=".1"
+          ixy="0.0"
+          ixz="0.0"
+          iyy=".1"
+          iyz="0.0"
+          izz=".1"/>
+      </inertial>
+    </link>
+  </xacro:macro>
   <gazebo>
     <!-- Freefloating gazebo plugin -->
     <plugin name="smtu_freefloating_gazebo_control"
-            filename="libsmtu_freefloating_gazebo_control.so">
+      filename="libsmtu_freefloating_gazebo_control.so">
       <switchService>switch</switchService>
       <updateRate>100</updateRate>
@@ -32,12 +57,4 @@
         <effort>30</effort>
       </thruster>
-    </plugin>
-    <plugin name="imu_plugin" filename="libgazebo_ros_imu.so">
-      <alwaysOn>true</alwaysOn>
-      <bodyName>base_link</bodyName>
-      <topicName>imu_data</topicName>
-      <serviceName>imu_service</serviceName>
-      <gaussianNoise>0.1</gaussianNoise>
-      <updateRate>10.0</updateRate>
     </plugin>
   </gazebo>
@@ -67,5 +84,5 @@
     </inertial>
     <buoyancy>
-      <variable/>
+      <compensation>1.0</compensation>
       <origin xyz= "0 0 0"/>
       <limit radius=".1"/>
@@ -73,3 +90,5 @@
     </buoyancy>
   </link>
+  <xacro:buoyancy_link name="front" xyz="-0.33 0 0"/>
+  <xacro:buoyancy_link name="rear" xyz="0.33 0 0"/>
 </robot>

Commit message: Changed visual model

File: urdf/uauv.xacro (robot description, xacro)
@@ -4,7 +4,7 @@
   <!-- Body properties -->
   <xacro:property name="body_mass"        value="10"/>
-  <xacro:property name="body_radius"      value="0.065"/>
-  <xacro:property name="body_length"      value="0.667"/>
-  <xacro:property name="X_cog"            value="-0.55"/>
+  <xacro:property name="body_radius"      value="0.05"/>
+  <xacro:property name="body_length"      value="1.163"/>
+  <xacro:property name="X_cog"            value="-0.45"/>
   <!-- Variable buoyancy link -->
   <xacro:macro name="buoyancy_link" params="name xyz">
@@ -67,7 +67,7 @@
     </visual>
     <collision>
-      <origin xyz="0 0 0" rpy="0 0 0"/>
+      <origin xyz="0 0 0" rpy="0 ${PI/2} 0"/>
       <geometry>
-        <mesh filename="package://smtu_uauv/objects/uauv.dae"/>
+        <cylinder radius="${body_radius}" length="${body_length}"/>
       </geometry>
     </collision>
@@ -90,5 +90,5 @@
     </buoyancy>
   </link>
-  <xacro:buoyancy_link name="front" xyz="-0.33 0 0"/>
-  <xacro:buoyancy_link name="rear" xyz="0.33 0 0"/>
+  <xacro:buoyancy_link name="front" xyz="-0.474 0 0"/>
+  <xacro:buoyancy_link name="rear" xyz="0.54 0 0"/>
 </robot>

Commit message: added uwsim support

File: urdf/uauv.xacro (robot description, xacro)
@@ -63,5 +63,5 @@
       <origin rpy="0 0 0" xyz="0 0 0"/>
       <geometry>
-        <mesh filename="package://smtu_uauv/objects/uauv.dae"/>
+        <mesh filename="package://smtu_uauv/objects/uauv.stl"/>
       </geometry>
     </visual>
